Commit message: controller for arm, draft

File: model/robot.urdf (robot description, URDF)
Before this commit: robot robot, 7 links, 6 joints
Links:
- added link left_wheel
- added link right_wheel
Joints:
- added joint wheel_left_joint: type continuous, parent base_link, child left_wheel
- added joint wheel_right_joint: type continuous, parent base_link, child right_wheel

Commit message: odometry multiplier tuned

File: model/robot.urdf (robot description, URDF)
Before this commit: robot robik, 9 links, 8 joints
Links:
- link clamp_link: geometry visual box size=0.02 0.08 0.01
