Commit message: befor hectorSLAM

File: model/v3/kinect.urdf.xacro (robot description, xacro)
@@ -2,10 +2,10 @@
 <robot name="sensor_kinect" xmlns:xacro="http://ros.org/wiki/xacro">
   <!-- Robik position -->
-  <property name="cam_px" value="-0.19" />
-  <property name="cam_py" value="0" />
-  <property name="cam_pz" value="0.59" />
-  <property name="cam_or" value="0" />
-  <property name="cam_op" value="0.262" />
-  <property name="cam_oy" value="0" />
+  <xacro:property name="cam_px" value="-0.19" />
+  <xacro:property name="cam_py" value="0" />
+  <xacro:property name="cam_pz" value="0.59" />
+  <xacro:property name="cam_or" value="0" />
+  <xacro:property name="cam_op" value="0.262" />
+  <xacro:property name="cam_oy" value="0" />
   <!--  <xacro:include filename="$(find robik)/model/v3/kinect_gazebo.urdf.xacro"/> -->
   <xacro:macro name="sensor_kinect" params="parent">

File: model/v3/robik.urdf.xacro (robot description, xacro)
@@ -1,5 +1,5 @@
 <?xml version="1.0"?>
 <!-- (x/red +dopredu -dozadu) (y/green -levo +vpravo) (z/blue -dolu +nahoru) -->
-<robot xmlns:xacro="http://www.ros.org/wiki/xacro" name="robik">
+<robot xmlns:xacro="http://ros.org/wiki/xacro" name="robik">
 	<!-- constants -->
 	<xacro:property name="pi" value="3.1415926535897931" />
