Commit message: grrr

File: model/v3/robik.urdf.xacro (robot description, xacro)
@@ -147,4 +147,14 @@
 		<xacro:antenna_templ y="-0.12" roll="0.1745" name_tmpl="right_backbone"/>
 	</link>
+	<joint name="base_footprint_joint" type="fixed">
+		<origin xyz="0 0 0" rpy="0 0 0" />
+		<parent link="base_footprint"/>
+		<child link="base_stabilized"/>
+	</joint>
+	<joint name="base_footprint_joint" type="fixed">
+		<origin xyz="0 0 0" rpy="0 0 0" />
+		<parent link="base_stabilized"/>
+		<child link="base_link"/>
+	</joint>
 	<!-- wheels -->
 	<xacro:macro name="wheel_templ">

Commit message: laser position bad

File: model/v3/robik.urdf.xacro (robot description, xacro)
@@ -78,5 +78,5 @@
 		<xacro:backbone_templ y="-0.07" name_tmpl="right_backbone"/>
 		<xacro:property name="head_base_templ">
-			<origin xyz="${-0.20 - 0.06/2 + 0.01/2} 0 ${backbone_length + base_above_gnd}" rpy="0 0 0" />
+			<origin xyz="-0.225 0 ${backbone_length + base_above_gnd}" rpy="0 0 0" />
 			<geometry>
 				<box size="0.06 0.22 0.02" />
@@ -147,4 +147,7 @@
 		<xacro:antenna_templ y="-0.12" roll="0.1745" name_tmpl="right_backbone"/>
 	</link>
+<!--
+	<link name="base_footprint" />
+	<link name="base_stabilized" />
 	<joint name="base_footprint_joint" type="fixed">
 		<origin xyz="0 0 0" rpy="0 0 0" />
@@ -152,9 +155,10 @@
 		<child link="base_stabilized"/>
 	</joint>
-	<joint name="base_footprint_joint" type="fixed">
+	<joint name="base_stabilized_joint" type="fixed">
 		<origin xyz="0 0 0" rpy="0 0 0" />
 		<parent link="base_stabilized"/>
 		<child link="base_link"/>
 	</joint>
+-->
 	<!-- wheels -->
 	<xacro:macro name="wheel_templ">

Commit message: odomtery fail

File: model/v3/robik.urdf.xacro (robot description, xacro)
@@ -8,5 +8,5 @@
 	<!-- measurements -->
 	<xacro:property name="base_above_gnd" value="0.065" />
-	<xacro:property name="base_lenght" value="0.365" />
+	<xacro:property name="base_length" value="0.365" />
 	<xacro:property name="base_width" value="0.352" />
 	<xacro:property name="wheel_radius" value="0.05" />
@@ -38,5 +38,5 @@
 			<origin xyz="-0.06 0 ${base_above_gnd}" rpy="0 0 0" />
 			<geometry>
-				<box size="${base_lenght} ${base_width} ${plastic_thickness}" />
+				<box size="${base_length} ${base_width} ${plastic_thickness}" />
 			</geometry>
 		</collision>
@@ -60,7 +60,7 @@
 			</geometry>
 		</collision>
-		<xacro:macro name="backbone_templ" params="y name_tmpl">
+		<xacro:macro name="backbone_templ" params="y name_tmpl origin_z">
 			<visual name="{$name_tmpl}_visual">
-				<origin xyz="-0.225 ${y} ${backbone_length / 2 + base_above_gnd}" rpy="0 0 0" />
+				<origin xyz="-0.225 ${y} ${origin_z}" rpy="0 0 0" />
 				<geometry>
 					<box size="0.01 0.01 ${backbone_length}" />
@@ -69,5 +69,5 @@
 			</visual>
 			<collision>
-				<origin xyz="-0.225 ${y} ${backbone_length / 2 + base_above_gnd}" rpy="0 0 0" />
+				<origin xyz="-0.225 ${y} ${origin_z}" rpy="0 0 0" />
 				<geometry>
 					<box size="0.01 0.01 ${backbone_length}" />
@@ -75,6 +75,6 @@
 			</collision>
 		</xacro:macro>
-		<xacro:backbone_templ y="0.07" name_tmpl="left_backbone"/>
-		<xacro:backbone_templ y="-0.07" name_tmpl="right_backbone"/>
+		<xacro:backbone_templ y="0.07" name_tmpl="left_backbone" origin_z="${backbone_length / 2 + base_above_gnd}" />
+		<xacro:backbone_templ y="-0.07" name_tmpl="right_backbone" origin_z="${backbone_length / 2 + base_above_gnd}" />
 		<xacro:property name="head_base_templ">
 			<origin xyz="-0.225 0 ${backbone_length + base_above_gnd}" rpy="0 0 0" />
@@ -206,4 +206,10 @@
 	<xacro:include filename="$(find robik)/model/v3/kinect.urdf.xacro"/>
 	<xacro:sensor_kinect parent="base_link" />
+	<link name="base_scan_link" />
+	<joint name="base_scan_joint" type="fixed">
+		<parent link="base_link" />
+		<child link="base_scan_link" />
+		<origin xyz="-0.19 0 0.59" rpy="0 0 0" />
+	</joint>
 	<!-- arm -->
 	<link name="yaw_link">

Commit message: xacro fix

File: model/v3/robik.urdf.xacro (robot description, xacro)
@@ -3,5 +3,5 @@
 <robot xmlns:xacro="http://ros.org/wiki/xacro" name="robik">
 	<!-- constants -->
-	<xacro:property name="pi" value="3.1415926535897931" />
+	<!--<xacro:property name="pi" value="3.1415926535897931" /> -->
 	<xacro:property name="pi_half" value="${pi /2}" />
 	<xacro:property name="plastic_thickness" value="0.006" />

Commit message: adding wiimote

File: model/v3/robik.urdf.xacro (robot description, xacro)
@@ -189,18 +189,4 @@
 		<child link="right_wheel"/>
 	</joint>
-	<link name="rear_sonar_link">
-		<visual>
-			<origin xyz="-0.015 0 0" rpy="0 0 0" />
-			<geometry>
-				<box size="0.03 0.04 0.015" />
-			</geometry>
-			<material name="alum" />
-		</visual>
-	</link>
-	<joint name="rear_sonar_joint" type="fixed">
-		<parent link="base_link" />
-		<child link="rear_sonar_link" />
-		<origin xyz="-0.24 0 ${0.015 + base_above_gnd}" rpy="0 0 ${pi}" />
-	</joint>
 	<!-- kinect -->
 	<xacro:include filename="$(find robik)/model/v3/kinect.urdf.xacro"/>

Commit message: lidar mounted

File: model/v3/robik.urdf.xacro (robot description, xacro)
@@ -196,5 +196,5 @@
 		<parent link="base_link" />
 		<child link="base_scan_link" />
-		<origin xyz="-0.19 0 0.59" rpy="0 0 0" />
+		<origin xyz="-0.15 0 0.15" rpy="0 0 0" />
 	</joint>
 	<!-- arm -->
