Commit message: preparation for open fair enode name="candy" pkg="robik" type="candy.py" />

File: model/v3/robik.urdf (robot description, URDF)
Before this commit: robot robik, 15 links, 14 joints
Links:
- link clamp_link: geometry visual box size=0.02 0.09 0.01

File: model/v3/robik.urdf.xacro (robot description, xacro)
@@ -270,7 +270,7 @@
 	<link name="clamp_link">
 		<visual>
-			<origin xyz="0 0.025 0" rpy="0 0 0"/>
-			<geometry>
-				<box size="0.02 0.05 0.01" />
+			<origin xyz="0 0.057 0" rpy="0 0 0"/>
+			<geometry>
+				<box size="0.02 0.09 0.01" />
 			</geometry>
 			<material name="alum">
