Commit message: urdf

File: src/robik_description/urdf/kinect.urdf.xacro (robot description, xacro)
@@ -8,5 +8,5 @@
   <xacro:property name="cam_op" value="0.262" />
   <xacro:property name="cam_oy" value="0" />
-  <!--  <xacro:include filename="$(find robik)/model/v3/kinect_gazebo.urdf.xacro"/> -->
+  <!--  <xacro:include filename="$(find robik_description)/urdf/kinect_gazebo.urdf.xacro"/> -->
   <xacro:macro name="sensor_kinect" params="parent">
     <joint name="camera_rgb_joint" type="fixed">

File: src/robik_description/urdf/robik.urdf (robot description, URDF)
Before this commit: robot robik, 15 links, 14 joints
Links:
- removed link rear_sonar_link
- link base_link: geometry collision box size=0.006 0.125 0.125; collision box size=0.006 0.22 0.15
Joints:
- removed joint rear_sonar_joint
- joint base_scan_joint: origin xyz=-0.19 0 0.59 rpy=0 0 0 -> xyz=-0.15 0 0.15 rpy=0 0 0

File: src/robik_description/urdf/robik.urdf.xacro (robot description, xacro)
@@ -24,5 +24,5 @@
 	</material>
 	<material name="jetson">
-		<texture filename="package://robik/model/v3/textures/jetson.jpg" />
+		<texture filename="package://robik_description/materials/jetson.jpg" />
 	</material>
 	<!-- base -->
@@ -31,5 +31,5 @@
 			<origin xyz="0 0 ${base_above_gnd}" rpy="0 0 0" />
 			<geometry>
-				<mesh filename="package://robik/model/v3/meshes/base-binary.stl" scale="1.0 1.0 1.0" />
+				<mesh filename="package://robik_description/meshes/base-binary.stl" scale="1.0 1.0 1.0" />
 			</geometry>
 			<material name="clear_plastic" />
@@ -190,5 +190,5 @@
 	</joint>
 	<!-- kinect -->
-	<xacro:include filename="$(find robik)/model/v3/kinect.urdf.xacro"/>
+	<xacro:include filename="$(find robik_description)/urdf/kinect.urdf.xacro"/>
 	<xacro:sensor_kinect parent="base_link" />
 	<link name="base_scan_link" />

Commit message: urdf diff controler

File: src/robik_description/urdf/kinect.urdf.xacro (robot description, xacro)
@@ -47,5 +47,5 @@
             <origin xyz="0 0 0" rpy="0 0 ${pi/2}"/>
             <geometry>
-              <mesh filename="package://robik/model/v3/meshes/kinect.dae"/>
+              <mesh filename="package://robik_description/meshes/kinect.dae"/>
             </geometry>
           </visual>

File: src/robik_description/urdf/robik.urdf (robot description, URDF)
Before this commit: robot robik, 14 links, 13 joints
Links:
- link base_link: mass None -> 5.3
- link camera_link: geometry collision box size=0.07271 0.27794 0.073; visual mesh filename=package://robik_description/meshes/kinect.dae
- link clamp_link: mass None -> 0.15
- link elbow_link: mass None -> 0.15
- link left_wheel: mass None -> 0.3
- link right_wheel: mass None -> 0.3
- link roll_link: mass None -> 0.15
- link shoulder_link: mass None -> 0.15
- link yaw_link: mass None -> 0.15

File: src/robik_description/urdf/robik.urdf.xacro (robot description, xacro)
@@ -13,17 +13,8 @@
 	<xacro:property name="wheel_distance" value="0.30" />
 	<xacro:property name="backbone_length" value="0.485" />
-	<!-- materials -->
-	<material name="clear_plastic">
-		<color rgba="0.81 0.81 0.81 0.5" />
-	</material>
-	<material name="alum">
-		<color rgba="0.81 0.88 0.91 1" />
-	</material>
-	<material name="wood">
-		<color rgba="1 0.81 0.4 1" />
-	</material>
-	<material name="jetson">
-		<texture filename="package://robik_description/materials/jetson.jpg" />
-	</material>
+  <!-- Import all Gazebo-customization elements, including Gazebo colors -->
+  <xacro:include filename="$(find robik_description)/urdf/robik.gazebo" />
+  <xacro:include filename="$(find robik_description)/urdf/materials.xacro" />
+  <xacro:include filename="$(find robik_description)/urdf/macros.xacro" />
 	<!-- base -->
 	<link name="base_link">
@@ -146,31 +137,14 @@
 		<xacro:antenna_templ y="0.12" roll="-0.1745" name_tmpl="left_backbone"/>
 		<xacro:antenna_templ y="-0.12" roll="0.1745" name_tmpl="right_backbone"/>
-	</link>
-<!--
-	<link name="base_footprint" />
-	<link name="base_stabilized" />
-	<joint name="base_footprint_joint" type="fixed">
-		<origin xyz="0 0 0" rpy="0 0 0" />
-		<parent link="base_footprint"/>
-		<child link="base_stabilized"/>
-	</joint>
-	<joint name="base_stabilized_joint" type="fixed">
-		<origin xyz="0 0 0" rpy="0 0 0" />
-		<parent link="base_stabilized"/>
-		<child link="base_link"/>
-	</joint>
--->
+		<inertial>
+			<origin xyz="0 0 0.1" rpy="0 0 0"/>
+			<mass value="5.3"/>
+			<inertia
+				ixx="1" ixy="0.0" ixz="0.0"
+				iyy="1" iyz="0.0"
+				izz="1"/>
+		</inertial>
+	</link>
 	<!-- wheels -->
-	<xacro:macro name="wheel_templ">
-		<visual>
-			<origin xyz="0 0 0" rpy="0 ${pi_half} ${pi_half}" />
-			<geometry>
-				<cylinder radius="${wheel_radius}" length="0.04" />
-			</geometry>
-			<material name="black_wheel">
-				<color rgba="0.1 0.1 0.1 1" />
-			</material>
-		</visual>
-	</xacro:macro>
 	<link name="left_wheel">
 		<xacro:wheel_templ/>
@@ -183,4 +157,5 @@
 		<parent link="base_link"/>
 		<child link="left_wheel"/>
+		<joint_properties damping="1.0" friction="1.0"/>
 	</joint>
 	<joint name="wheel_right_joint" type="continuous">
@@ -188,4 +163,5 @@
 		<parent link="base_link"/>
 		<child link="right_wheel"/>
+		<joint_properties damping="1.0" friction="1.0"/>
 	</joint>
 	<!-- kinect -->
@@ -199,4 +175,14 @@
 	</joint>
 	<!-- arm -->
+	<xacro:macro name="arm_inertia_templ">
+		<inertial>
+			<origin xyz="0 0 0.1" rpy="0 0 0"/>
+			<mass value="0.15"/>
+			<inertia
+				ixx="1" ixy="0.0" ixz="0.0"
+				iyy="1" iyz="0.0"
+				izz="1"/>
+		</inertial>
+	</xacro:macro>
 	<link name="yaw_link">
 		<visual>
@@ -207,4 +193,5 @@
 			<material name="wood" />
 		</visual>
+		<xacro:arm_inertia_templ/>
 	</link>
 	<joint name="yaw_joint" type="revolute">
@@ -214,4 +201,5 @@
 		<axis xyz="0 0 -1" />
 		<limit lower="-1.8675023" upper="1.099557429" effort="1000" velocity="1" />
+		<dynamics damping="0.7"/>
 	</joint>
 	<link name="shoulder_link">
@@ -225,4 +213,5 @@
 			</material>
 		</visual>
+		<xacro:arm_inertia_templ/>
 	</link>
 	<joint name="shoulder_joint" type="revolute">
@@ -232,4 +221,5 @@
 		<axis xyz="1 0 0" />
 		<limit lower="0" upper="2.094395102" effort="1000" velocity="1" />
+		<dynamics damping="0.7"/>
 	</joint>
 	<link name="elbow_link">
@@ -243,4 +233,5 @@
 			</material>
 		</visual>
+		<xacro:arm_inertia_templ/>
 	</link>
 	<joint name="elbow_joint" type="revolute">
@@ -250,4 +241,5 @@
 		<axis xyz="1 0 0" />
 		<limit lower="-1.919862177" upper="0.6981317008" effort="1000" velocity="1" />
+		<dynamics damping="0.7"/>
 	</joint>
 	<link name="roll_link">
@@ -260,4 +252,5 @@
 			</material>
 		</visual>
+		<xacro:arm_inertia_templ/>
 	</link>
 	<joint name="roll_joint" type="revolute">
@@ -267,4 +260,5 @@
 		<axis xyz="0 1 0" />
 		<limit lower="-1.570796327" upper="1.570796327" effort="1000" velocity="1" />
+		<dynamics damping="0.7"/>
 	</joint>
 	<link name="clamp_link">
@@ -278,4 +272,5 @@
 			</material>
 		</visual>
+		<xacro:arm_inertia_templ/>
 	</link>
 	<joint name="clamp_joint" type="revolute">
@@ -286,4 +281,5 @@
 		<limit lower="0" upper="0.6981317008" effort="1000" velocity="1" />
 		<!--<mimic joint="clamp_joint" multiplier="-1" offset="0"/>-->
+		<dynamics damping="0.7"/>
 	</joint>
 </robot>
