Commit message: roscontrol loads

File: src/robik_description/urdf/macros.xacro (robot description, xacro)
@@ -11,4 +11,10 @@
 			</material>
 		</visual>
+		<collision>
+			<origin xyz="0 0 0" rpy="0 ${pi_half} ${pi_half}" />
+			<geometry>
+				<cylinder radius="${wheel_radius}" length="0.04" />
+			</geometry>
+		</collision>
 		<inertial>
 			<origin xyz="0 0 0.1" rpy="0 0 0"/>
@@ -20,3 +26,13 @@
 		</inertial>
 	</xacro:macro>
+	<xacro:macro name="arm_inertia_templ">
+		<inertial>
+			<origin xyz="0 0 0.1" rpy="0 0 0"/>
+			<mass value="0.15"/>
+			<inertia
+				ixx="1" ixy="0.0" ixz="0.0"
+				iyy="1" iyz="0.0"
+				izz="1"/>
+		</inertial>
+	</xacro:macro>
 </robot>

File: src/robik_description/urdf/robik.urdf.xacro (robot description, xacro)
@@ -18,4 +18,5 @@
   <xacro:include filename="$(find robik_description)/urdf/macros.xacro" />
 	<!-- base -->
+	<link name="dummy" />
 	<link name="base_link">
 		<visual name="base">
@@ -146,4 +147,8 @@
 		</inertial>
 	</link>
+    <joint name="dummy_joint" type="fixed">
+     <parent link="dummy"/>
+     <child link="base_link"/>
+   </joint>
 	<!-- wheels -->
 	<link name="left_wheel">
@@ -154,5 +159,5 @@
 	</link>
 	<joint name="wheel_left_joint" type="continuous">
-		<origin xyz="0 ${wheel_distance / 2} ${wheel_radius}" rpy="0 0 0" />
+		<origin xyz="0 ${wheel_distance / 2} ${wheel_radius}" rpy="1 0 0" />
 		<parent link="base_link"/>
 		<child link="left_wheel"/>
@@ -160,9 +165,29 @@
 	</joint>
 	<joint name="wheel_right_joint" type="continuous">
-		<origin xyz="0 -${wheel_distance / 2} ${wheel_radius}" rpy="0 0 0" />
+		<origin xyz="0 -${wheel_distance / 2} ${wheel_radius}" rpy="1 0 0" />
 		<parent link="base_link"/>
 		<child link="right_wheel"/>
 		<joint_properties damping="1.0" friction="1.0"/>
 	</joint>
+	<transmission name="tran_wheel_left_joint">
+		<type>transmission_interface/SimpleTransmission</type>
+		<joint name="wheel_left_joint">
+			<hardwareInterface>hardware_interface/VelocityJointInterface</hardwareInterface>
+		</joint>
+		<actuator name="motor_wheel_left_joint">
+			<hardwareInterface>hardware_interface/VelocityJointInterface</hardwareInterface>
+			<mechanicalReduction>1</mechanicalReduction>
+		</actuator>
+	</transmission>
+	<transmission name="tran_wheel_right_joint">
+		<type>transmission_interface/SimpleTransmission</type>
+		<joint name="wheel_right_joint">
+			<hardwareInterface>hardware_interface/VelocityJointInterface</hardwareInterface>
+		</joint>
+		<actuator name="motor_wheel_right_joint">
+			<hardwareInterface>hardware_interface/VelocityJointInterface</hardwareInterface>
+			<mechanicalReduction>1</mechanicalReduction>
+		</actuator>
+	</transmission>
 	<!-- kinect -->
 	<xacro:include filename="$(find robik_description)/urdf/kinect.urdf.xacro"/>
@@ -175,14 +200,4 @@
 	</joint>
 	<!-- arm -->
-	<xacro:macro name="arm_inertia_templ">
-		<inertial>
-			<origin xyz="0 0 0.1" rpy="0 0 0"/>
-			<mass value="0.15"/>
-			<inertia
-				ixx="1" ixy="0.0" ixz="0.0"
-				iyy="1" iyz="0.0"
-				izz="1"/>
-		</inertial>
-	</xacro:macro>
 	<link name="yaw_link">
 		<visual>
@@ -193,4 +208,10 @@
 			<material name="wood" />
 		</visual>
+		<collision>
+			<origin xyz="0 0 ${0.06 / 2}" rpy="0 0 0" />
+			<geometry>
+				<box size="0.045 0.04 0.06" />
+			</geometry>
+		</collision>
 		<xacro:arm_inertia_templ/>
 	</link>

Commit message: inertia and wheel link fixed

File: src/robik_description/urdf/macros.xacro (robot description, xacro)
@@ -7,7 +7,5 @@
 				<cylinder radius="${wheel_radius}" length="0.04" />
 			</geometry>
-			<material name="black_wheel">
-				<color rgba="0.1 0.1 0.1 1" />
-			</material>
+			<material name="jetson" />
 		</visual>
 		<collision>

File: src/robik_description/urdf/robik.urdf.xacro (robot description, xacro)
@@ -139,5 +139,5 @@
 		<xacro:antenna_templ y="-0.12" roll="0.1745" name_tmpl="right_backbone"/>
 		<inertial>
-			<origin xyz="0 0 0.1" rpy="0 0 0"/>
+			<origin xyz="-0.1 0 0.1" rpy="0 0 0"/>
 			<mass value="5.3"/>
 			<inertia
@@ -159,13 +159,15 @@
 	</link>
 	<joint name="wheel_left_joint" type="continuous">
-		<origin xyz="0 ${wheel_distance / 2} ${wheel_radius}" rpy="1 0 0" />
-		<parent link="base_link"/>
-		<child link="left_wheel"/>
+		<origin xyz="0 ${wheel_distance / 2} ${wheel_radius}" rpy="0 0 0" />
+		<parent link="base_link" />
+		<child link="left_wheel" />
+		<axis xyz="0 0 1" />
 		<joint_properties damping="1.0" friction="1.0"/>
 	</joint>
 	<joint name="wheel_right_joint" type="continuous">
-		<origin xyz="0 -${wheel_distance / 2} ${wheel_radius}" rpy="1 0 0" />
+		<origin xyz="0 -${wheel_distance / 2} ${wheel_radius}" rpy="0 0 0" />
 		<parent link="base_link"/>
 		<child link="right_wheel"/>
+		<axis xyz="0 0 1" />
 		<joint_properties damping="1.0" friction="1.0"/>
 	</joint>
@@ -234,4 +236,10 @@
 			</material>
 		</visual>
+		<collision>
+			<origin xyz="0 0.0675 0" rpy="0 0 0"/>
+			<geometry>
+				<box size="0.04 0.135 0.02" />
+			</geometry>
+		</collision>
 		<xacro:arm_inertia_templ/>
 	</link>
@@ -250,8 +258,12 @@
 				<box size="0.04 0.065 0.02" />
 			</geometry>
-			<material name="wood">
-				<color rgba="0 1.0 1.0 1.0" />
-			</material>
-		</visual>
+			<material name="wood" />
+		</visual>
+		<collision>
+			<origin xyz="0 0.0325 0" rpy="0 0 0"/>
+			<geometry>
+				<box size="0.04 0.065 0.02" />
+			</geometry>
+		</collision>
 		<xacro:arm_inertia_templ/>
 	</link>
@@ -269,8 +281,11 @@
 				<box size="0.03 0.003 0.04" />
 			</geometry>
-			<material name="wood">
-				<color rgba="0 1.0 1.0 1.0" />
-			</material>
-		</visual>
+			<material name="wood" />
+		</visual>
+		<collision>
+			<geometry>
+				<box size="0.03 0.003 0.04" />
+			</geometry>
+		</collision>
 		<xacro:arm_inertia_templ/>
 	</link>
@@ -289,8 +304,12 @@
 				<box size="0.02 0.09 0.01" />
 			</geometry>
-			<material name="alum">
-				<color rgba="0 1.0 1.0 1.0" />
-			</material>
-		</visual>
+			<material name="alum" />
+		</visual>
+		<collision>
+			<origin xyz="0 0.057 0" rpy="0 0 0"/>
+			<geometry>
+				<box size="0.02 0.09 0.01" />
+			</geometry>
+		</collision>
 		<xacro:arm_inertia_templ/>
 	</link>
